File: PCB/Tiebox.kicad_pcb (KiCad board)
At the start: 2 copper layers, 304 x 149 mm, 64 parts, among them J1 USB C Connector, J2 JTAG_TC2030, SW1 Boot, U1 XC6206, U2 USBLC6-2SC6, U3 RP2040, U4 W25Q128JVS, Y1 12MHz

Commit message: v1
Parts:
- added CH1: choc_v1_SW_HS, PCM_marbastlib-choc:SW_choc_v1_HS_CPG135001S30_1u, B.Cu at (36.8, 157.6)
- added CH10: choc_v1_SW_HS, PCM_marbastlib-choc:SW_choc_v1_HS_CPG135001S30_1u, B.Cu at (231.1, 163.0)
- added CH11: choc_v1_SW_HS, PCM_marbastlib-choc:SW_choc_v1_HS_CPG135001S30_1u, B.Cu at (254.5, 147.8)
- added CH12: choc_v1_SW_HS, PCM_marbastlib-choc:SW_choc_v1_HS_CPG135001S30_1u, B.Cu at (281.5, 146.5)
- added CH13: choc_v1_SW_HS, PCM_marbastlib-choc:SW_choc_v1_HS_CPG135001S30_1u, B.Cu at (308.4, 157.6)
- added CH14: choc_v1_SW_HS, PCM_marbastlib-choc:SW_choc_v1_HS_CPG135001S30_1u, B.Cu at (129.0, 219.9)
- added CH15: choc_v1_SW_HS, PCM_marbastlib-choc:SW_choc_v1_HS_CPG135001S30_1u, B.Cu at (147.8, 238.0)
- added CH16: choc_v1_SW_HS, PCM_marbastlib-choc:SW_choc_v1_HS_CPG135001S30_1u, B.Cu at (197.4, 238.0)
- added CH17: choc_v1_SW_HS, PCM_marbastlib-choc:SW_choc_v1_HS_CPG135001S30_1u, B.Cu at (216.3, 219.9)
- added CH18: choc_v1_SW_HS, PCM_marbastlib-choc:SW_choc_v1_HS_CPG135001S30_1u, B.Cu at (235.6, 201.9)
- added CH19: choc_v1_SW_HS, PCM_marbastlib-choc:SW_choc_v1_HS_CPG135001S30_1u, B.Cu at (192.8, 208.7)
- added CH2: choc_v1_SW_HS, PCM_marbastlib-choc:SW_choc_v1_HS_CPG135001S30_1u, B.Cu at (63.8, 146.5)
- added CH20: choc_v1_SW_HS, PCM_marbastlib-choc:SW_choc_v1_HS_CPG135001S30_1u, B.Cu at (212.1, 190.6)
- added CH3: choc_v1_SW_HS, PCM_marbastlib-choc:SW_choc_v1_HS_CPG135001S30_1u, B.Cu at (90.8, 147.8)
- added CH4: choc_v1_SW_HS, PCM_marbastlib-choc:SW_choc_v1_HS_CPG135001S30_1u, B.Cu at (114.1, 163.0)
- added CH5: choc_v1_SW_HS, PCM_marbastlib-choc:SW_choc_v1_HS_CPG135001S30_1u, B.Cu at (172.6, 163.0)
- added CH6: choc_v1_SW_HS, PCM_marbastlib-choc:SW_choc_v1_HS_CPG135001S30_1u, B.Cu at (227.1, 137.2)
- added CH7: choc_v1_SW_HS, PCM_marbastlib-choc:SW_choc_v1_HS_CPG135001S30_1u, B.Cu at (250.6, 122.0)
- added CH8: choc_v1_SW_HS, PCM_marbastlib-choc:SW_choc_v1_HS_CPG135001S30_1u, B.Cu at (277.3, 120.6)
- added CH9: choc_v1_SW_HS, PCM_marbastlib-choc:SW_choc_v1_HS_CPG135001S30_1u, B.Cu at (304.2, 131.7)
- added G***: LOGO, LOGO, B.Cu at (72.6, 166.7)
- added H5: MountingHole, qw-logo:qw new logo silk + copper md, F.Cu at (200.0, 117.9)
- added H6: MountingHole, qw-logo:qw new logo silk + copper md, B.Cu at (315.5, 175.0)
- added H7: MountingHole, 1999:1999 logo md, F.Cu at (23.8, 176.2)
- added H8: MountingHole, 1999:1999 logo md, B.Cu at (240.5, 240.5)
- added J3: Conn_01x04, Connector_PinHeader_2.54mm:PinHeader_1x04_P2.54mm_Vertical, F.Cu at (129.3, 140.5)
Connections:
- MX1 pad 1: unconnected-(MX1-Pad1) -> L
- MX1 pad 2: unconnected-(MX1-Pad2) -> GND
- MX10 pad 1: unconnected-(MX10-Pad1) -> B
- MX10 pad 2: unconnected-(MX10-Pad2) -> GND
- MX11 pad 1: unconnected-(MX11-Pad1) -> X
- MX11 pad 2: unconnected-(MX11-Pad2) -> GND
- MX12 pad 1: unconnected-(MX12-Pad1) -> Z
- MX12 pad 2: unconnected-(MX12-Pad2) -> GND
- MX13 pad 1: unconnected-(MX13-Pad1) -> UP
- MX13 pad 2: unconnected-(MX13-Pad2) -> GND
- MX14 pad 1: unconnected-(MX14-Pad1) -> M1
- MX14 pad 2: unconnected-(MX14-Pad2) -> GND
- MX15 pad 1: unconnected-(MX15-Pad1) -> M2
- MX15 pad 2: unconnected-(MX15-Pad2) -> GND
- MX16 pad 1: unconnected-(MX16-Pad1) -> C_DN
- MX16 pad 2: unconnected-(MX16-Pad2) -> GND
- MX17 pad 1: unconnected-(MX17-Pad1) -> A
- MX17 pad 2: unconnected-(MX17-Pad2) -> GND
- MX18 pad 1: unconnected-(MX18-Pad1) -> C_RT
- MX18 pad 2: unconnected-(MX18-Pad2) -> GND
- MX19 pad 1: unconnected-(MX19-Pad1) -> C_LT
- MX19 pad 2: unconnected-(MX19-Pad2) -> GND
- MX2 pad 1: unconnected-(MX2-Pad1) -> LEFT
- MX2 pad 2: unconnected-(MX2-Pad2) -> GND
- MX20 pad 1: unconnected-(MX20-Pad1) -> C_UP
- MX20 pad 2: unconnected-(MX20-Pad2) -> GND
- MX3 pad 1: unconnected-(MX3-Pad1) -> DOWN
- MX3 pad 2: unconnected-(MX3-Pad2) -> GND
- MX4 pad 1: unconnected-(MX4-Pad1) -> RIGHT
- MX4 pad 2: unconnected-(MX4-Pad2) -> GND
- MX5 pad 1: unconnected-(MX5-Pad1) -> START
- MX5 pad 2: unconnected-(MX5-Pad2) -> GND
- MX6 pad 1: unconnected-(MX6-Pad1) -> R
- MX6 pad 2: unconnected-(MX6-Pad2) -> GND
- MX7 pad 1: unconnected-(MX7-Pad1) -> Y
- MX7 pad 2: unconnected-(MX7-Pad2) -> GND
- MX8 pad 1: unconnected-(MX8-Pad1) -> LS
- MX8 pad 2: unconnected-(MX8-Pad2) -> GND
- MX9 pad 1: unconnected-(MX9-Pad1) -> MS
- MX9 pad 2: unconnected-(MX9-Pad2) -> GND
- U3 pad 11: unconnected-(U3-GPIO8-Pad11) -> SDA
- U3 pad 12: unconnected-(U3-GPIO9-Pad12) -> SCL
Routing:
- net C_DN: track 15.1 -> 203.3 mm
- net MS: track 15.9 -> 202.2 mm
- net L: track 17.3 -> 192.7 mm
- net LS: track 14.8 -> 185.7 mm
- net UP: track 16.4 -> 181.5 mm
- net C_LT: track 16.5 -> 177.9 mm
- net LEFT: track 17.3 -> 176.6 mm
- net A: track 16.0 -> 166.0 mm
- net Z: track 15.9 -> 164.2 mm
- net M1: track 17.2 -> 160.4 mm
- net Y: track 15.5 -> 158.1 mm
- net DOWN: track 16.9 -> 147.8 mm
- net M2: track 18.6 -> 141.9 mm
- net X: track 14.9 -> 134.9 mm
- net C_RT: track 17.0 -> 121.8 mm
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Other:
- outline, holes or cut-outs redrawn
- board text added: "GND 3v3 SCL SDA"
