File: PCB/Tiebox.kicad_sch (KiCad schematic)
At the start: 64 parts, among them J1 USB C Connector, J2 JTAG_TC2030, SW1 Boot, U1 XC6206, U2 USBLC6-2SC6, U3 RP2040, U4 W25Q128JVS, Y1 12MHz

Commit message: v1
Parts:
- added CH1, CH10, CH11, CH12, CH13, CH14, CH15, CH16, CH17, CH18, CH19, CH2, CH20, CH3, CH4, CH5, CH6, CH7, CH8, CH9: choc_v1_SW_HS, PCM_marbastlib-choc:SW_choc_v1_HS_CPG135001S30_1u, symbol PCM_marbastlib-choc:choc_v1_SW_HS_CPG135001S30
- added H5, H6: MountingHole, qw-logo:qw new logo silk + copper md, symbol Mechanical:MountingHole
- added H7, H8: MountingHole, 1999:1999 logo md, symbol Mechanical:MountingHole
- added J3: Conn_01x04, Connector_PinHeader_2.54mm:PinHeader_1x04_P2.54mm_Vertical, symbol Connector_Generic:Conn_01x04
Connections:
- net +3V3: now also J3.2 (Pin_2)
- net A: now also MX17.1, CH17.1
- net B: now also MX10.1, CH10.1
- net C_DN: now also MX16.1, CH16.1
- net C_LT: now also MX19.1, CH19.1
- net C_RT: now also MX18.1, CH18.1
- net C_UP: now also MX20.1, CH20.1
- net DOWN: now also MX3.1, CH3.1
- net GND: now also MX1.2, MX10.2, MX11.2, MX12.2, MX13.2, MX14.2, MX15.2, MX16.2, MX17.2, MX18.2, MX19.2, MX2.2, MX20.2, MX3.2, MX4.2, MX5.2, MX6.2, MX7.2, MX8.2, MX9.2, CH1.2, CH10.2, CH11.2, CH12.2, CH13.2, CH14.2, CH15.2, CH16.2, CH17.2, CH18.2, CH19.2, CH2.2, CH20.2, CH3.2, CH4.2, CH5.2, CH6.2, CH7.2, CH8.2, CH9.2, J3.1 (Pin_1)
- net L: now also MX1.1, CH1.1
- net LEFT: now also MX2.1, CH2.1
- net LS: now also MX8.1, CH8.1
- net M1: now also MX14.1, CH14.1
- net M2: now also MX15.1, CH15.1
- net MS: now also MX9.1, CH9.1
- net R: now also MX6.1, CH6.1
- net RIGHT: now also MX4.1, CH4.1
- net START: now also MX5.1, CH5.1
- net UP: now also MX13.1, CH13.1
- net X: now also MX11.1, CH11.1
- net Y: now also MX7.1, CH7.1
- net Z: now also MX12.1, CH12.1
- net SDA: now reaches U3.11 (GPIO8)
- net SDA: now also J3.4 (Pin_4)
- net SCL: now reaches U3.12 (GPIO9)
- net SCL: now also J3.3 (Pin_3)
- no-connect marks 11 -> 9
Other:
- moved on the sheet: H1, H2, H3, H4
